File: prime_modulate.kicad_pcb (KiCad board)
At the start: 2 copper layers, 166.5 x 135 mm, 115 parts, among them U1 CartBus, U2 CartBus

Commit message: Changed board outline
Parts:
- removed REF**: OLED_128x32, ScottoKeebs_Components:OLED_128x32
- added U?: RP2040_Zero, ScottoKeebs_MCU:RP2040_Zero, F.Cu at (245.3, 111.1)
- moved D56 64.1 mm to (287.4, 166.5), turned to 120 degrees
- moved D54 62.2 mm to (292.1, 192.9), turned to 30 degrees
- moved D55 44.1 mm to (304.0, 157.3), turned to 120 degrees
- moved S56 19.1 mm to (280.4, 165.5)
- moved S53 19.1 mm to (309.8, 176.9)
- moved S55 19.0 mm to (296.9, 155.9)
- moved S54 19.0 mm to (293.3, 186.4)
- moved D53 17.2 mm to (308.9, 183.4), turned to 30 degrees
- moved D17 0.06 mm to (174.0, 129.9)
- moved S5 0.06 mm to (168.3, 87.1)
- moved D11 0.06 mm to (174.0, 110.8)
- moved D5 0.06 mm to (174.0, 91.8)
- moved S11 0.06 mm to (168.3, 106.2)
- moved S17 0.06 mm to (168.3, 125.2)
- moved D23 0.06 mm to (174.0, 149.0)
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Other:
- board size 166.5 x 135 mm -> 168.4 x 140 mm
